File: hardware/VCAT-LightingPCB/canopyBoard/canopyBoard/ESP32.kicad_sch (KiCad schematic)
At the start: 21 parts, among them J3 USB_C_Receptacle_USB2.0_16P, SW3 BOOT Switch, SW4 RESET Button, U2 ESP32-C6-MINI-1

Commit message: added current check, please dont overwrite my file again
Parts:
- renumbered C20 to C1, C21 to C2, C22 to C3, C23 to C4, D5 to D1, D6 to D2, D7 to D3, D8 to D4, D9 to D5, J3 to J4, R11 to R1, R12 to R2, R13 to R3, R14 to R4, R15 to R5, R16 to R6, R17 to R7, R18 to R8, SW3 to SW1, SW4 to SW2, U2 to U1
