File: hardware/VCAT-LightingPCB/canopyBoard/canopyBoard/canopyBoard.kicad_sch (KiCad schematic)
At the start: 9 parts, among them J1 Conn_02x03_Counter_Clockwise, J12 CAN_DEBUG_NANO_01x04, J13 CAN_NANO_01x05, J14 CAN_NANO_01x05, J2 Conn_02x01, J3 Conn_02x01, J5 Conn_02x01

Commit message: please no overrides, complete with bus, hopefully
Parts:
- removed J12: CAN_DEBUG_NANO_01x04, LHRS_Connectors:Molex_Nano-Fit_105309-xx05_1x04_P2.50mm_Vertical, symbol lhrs_connectors:CAN_DEBUG_NANO_01x04
- added J6: CAN_DEBUG_NANO_01x04, LHRS_Connectors:Molex_Nano-Fit_105309-xx05_1x04_P2.50mm_Vertical, symbol lhrs_connectors:CAN_DEBUG_NANO_01x04
Connections:
- net CAN_H: now also J6.2 (CAN_H)
- net CAN_L: now also J6.3 (CAN_L)
- net GND: now also J6.4 (GND)
- net V_IN: now also J6.1 (12V)
Other:
- sheet Current Check ports: added {CURR}; removed BRK_CURR, LEFT_CURR, RIGHT_CURR, STROBE_CURR
- sheet Fet Logic ports: added {FET}, {SIG}; removed BRK_FET1, BRK_FET2, BRK_FET3, BRK_SIG, LEFT_FET, LEFT_SIG, RIGHT_FET, RIGHT_SIG, STROBE_FET, STROBE_SIG
- sheet MCU ports: added {CURR}, {SIG}; removed BRK_CURR, BRK_SIG, LEFT_CURR, LEFT_SIG, RIGHT_CURR, RIGHT_SIG, STROBE_CURR, STROBE_SIG
- note removed: "FET Logic"
- note removed: "Output 12V"
- note removed: "Output MCU"
- moved on the sheet: J1, J13, J14, J2, J3, J5, R41, R42
