File: hardware/VCAT-LightingPCB/canopyBoard/canopyBoard/canopyBoard.kicad_sch (KiCad schematic)
At the start: 9 parts, among them J1 Conn_02x03_Counter_Clockwise, J13 CAN_NANO_01x05, J14 CAN_NANO_01x05, J2 Conn_02x01, J3 Conn_02x01, J5 Conn_02x01, J6 CAN_DEBUG_NANO_01x04

Commit message: workday, fixed connector logic
Parts:
- removed J1: Conn_02x03_Counter_Clockwise, Package_SO:SOIC-8_3.9x4.9mm_P1.27mm, symbol Connector_Generic:Conn_02x03_Counter_Clockwise
- removed J2, J3, J5: Conn_02x01, Package_SO:SOIC-8_3.9x4.9mm_P1.27mm, symbol Connector_Generic:Conn_02x01
- added J10, J11, J12: Conn_02x02_Counter_Clockwise, Package_SO:SOIC-8_3.9x4.9mm_P1.27mm, symbol Connector_Generic:Conn_02x02_Counter_Clockwise
Connections:
- net LEFT_12V: now also J10.1 (Pin_1)
- net RIGHT_12V: now also J11.1 (Pin_1)
- new net CPY_12V: J12.1 (Pin_1)
- new net CPY_PWM: J12.4 (Pin_4)
- new net CPY_PWRFET: J12.2 (Pin_2)
- new net L_PWM: J10.4 (Pin_4)
- new net L_PWRFET: J10.2 (Pin_2)
- new net R_PWM: J11.4 (Pin_4)
- new net R_PWRFET: J11.2 (Pin_2)
- new net STRB_PWM: J12.3 (Pin_3)
- no-connect marks 0 -> 2
Other:
- sheet Current Check ports: added CPY_12V; removed BRK_12V, STROBE_12V
- sheet MCU ports: added {PWM}; removed none
- note removed: "BPS Strobe Custom Flex PCB"
- note removed: "LED Strips COmpatible with COTs"
- moved on the sheet: J13, J14, J6, R41, R42
