File: hardware/VCAT-LightingPCB/canopyBoard/canopyBoard/canopyBoard.kicad_sch (KiCad schematic)
At the start: 7 parts, among them J10 Conn_02x02_Counter_Clockwise, J11 Conn_02x02_Counter_Clockwise, J12 Conn_02x02_Counter_Clockwise, J2 CAN_NANO_01x05, J3 CAN_NANO_01x05, J7 DEBUG_CAN

Commit message: Untrack KiCad .history, convert KiCAD-Sharepoint to a submodule, remove LightsPCB
Other:
- sheet CAN_Transceiver1 renamed CAN_Transceiver
Changed lines of the file:
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@@
 	(text "Debug Conn\n"
 		(exclude_from_sim no)
-		(at 27.178 50.8 0)
+		(at 26.67 50.8 0)
 		(effects
 			(font
@@
 	(text "CAN BUS\n"
 		(exclude_from_sim no)
-		(at 26.416 14.986 0)
+		(at 26.67 15.24 0)
 		(effects
 			(font
@@
 	(text "LIGHTING STRIPS"
 		(exclude_from_sim no)
-		(at 30.734 81.534 0)
+		(at 30.48 81.28 0)
 		(effects
 			(font
@@
 	)
 	(junction
+		(at 102.87 34.29)
+		(diameter 0)
+		(color 0 0 0 0)
+	)
+	(junction
 		(at 149.86 91.44)
 		(diameter 0)
@@
 	)
 	(junction
-		(at 171.45 68.58)
+		(at 171.45 67.31)
 		(diameter 0)
 		(color 0 0 0 0)
@@
 	(wire
 		(pts
+			(xy 102.87 34.29) (xy 100.33 34.29)
+		)
+		(stroke
+			(width 0)
+			(type default)
+		)
+	)
+	(wire
+		(pts
 			(xy 148.59 29.21) (xy 148.59 34.29)
 		)
@@
 	(wire
 		(pts
+			(xy 171.45 67.31) (xy 171.45 68.58)
+		)
+		(stroke
+			(width 0)
+			(type default)
+		)
+	)
+	(wire
+		(pts
 			(xy 44.45 113.03) (xy 45.72 113.03)
 		)
@@
 	(wire
 		(pts
-			(xy 110.49 34.29) (xy 100.33 34.29)
+			(xy 110.49 34.29) (xy 102.87 34.29)
 		)
 		(stroke
@@
 	(wire
 		(pts
-			(xy 170.18 67.31) (xy 171.45 68.58)
-		)
-		(stroke
-			(width 0)
-			(type default)
-		)
-	)
-	(wire
-		(pts
 			(xy 44.45 111.76) (xy 44.45 113.03)
 		)
@@
 	(wire
 		(pts
-			(xy 167.64 67.31) (xy 170.18 67.31)
+			(xy 167.64 67.31) (xy 171.45 67.31)
 		)
 		(stroke
@@
 	(symbol
 		(lib_id "power:PWR_FLAG")
-		(at 171.45 68.58 0)
+		(at 171.45 67.31 0)
 		(unit 1)
 		(body_style 1)
@@
 		(fields_autoplaced yes)
 		(property "Reference" "#FLG02"
-			(at 171.45 66.675 0)
+			(at 171.45 65.405 0)
 			(hide yes)
 			(show_name no)
@@
 		)
 		(property "Value" "PWR_FLAG"
-			(at 171.45 63.5 0)
+			(at 171.45 62.23 0)
 			(hide yes)
 			(show_name no)
@@
 		)
 		(property "Footprint" ""
-			(at 171.45 68.58 0)
+			(at 171.45 67.31 0)
 			(hide yes)
 			(show_name no)
@@
 		)
 		(property "Datasheet" ""
-			(at 171.45 68.58 0)
+			(at 171.45 67.31 0)
 			(hide yes)
 			(show_name no)
@@
 		)
 		(property "Description" "Special symbol for telling ERC where power comes from"
-			(at 171.45 68.58 0)
+			(at 171.45 67.31 0)
 			(hide yes)
 			(show_name no)
@@
 	)
 	(symbol
+		(lib_id "power:PWR_FLAG")
+		(at 102.87 34.29 0)
+		(unit 1)
+		(body_style 1)
+		(exclude_from_sim no)
+		(in_bom yes)
+		(on_board yes)
+		(in_pos_files yes)
+		(dnp no)
+		(fields_autoplaced yes)
+		(property "Reference" "#FLG012"
+			(at 102.87 32.385 0)
+			(hide yes)
+			(show_name no)
+			(do_not_autoplace no)
+			(effects
+				(font
+					(size 1.27 1.27)
+				)
+			)
+		)
+		(property "Value" "PWR_FLAG"
+			(at 102.87 29.21 0)
+			(hide yes)
+			(show_name no)
+			(do_not_autoplace no)
+			(effects
+				(font
+					(size 1.27 1.27)
+				)
+			)
+		)
+		(property "Footprint" ""
+			(at 102.87 34.29 0)
+			(hide yes)
+			(show_name no)
+			(do_not_autoplace no)
+			(effects
+				(font
+					(size 1.27 1.27)
+				)
+			)
+		)
+		(property "Datasheet" ""
+			(at 102.87 34.29 0)
+			(hide yes)
+			(show_name no)
+			(do_not_autoplace no)
+			(effects
+				(font
+					(size 1.27 1.27)
+				)
+			)
+		)
+		(property "Description" "Special symbol for telling ERC where power comes from"
+			(at 102.87 34.29 0)
+			(hide yes)
+			(show_name no)
+			(do_not_autoplace no)
+			(effects
+				(font
+					(size 1.27 1.27)
+				)
+			)
+		)
+		(pin "1"
+		)
+		(instances
+			(project "canopyBoard"
+				(path "/df5034a6-89e6-4596-8ae4-d16cb76dc299"
+					(reference "#FLG012")
+					(unit 1)
+				)
+			)
+		)
+	)
+	(symbol
 		(lib_id "power:GND")
 		(at 144.78 43.18 0)
@@
 			(color 0 0 0 0)
 		)
-		(property "Sheetname" "CAN_Transceiver1"
+		(property "Sheetname" "CAN_Transceiver"
 			(at 147.32 56.642 0)
 			(show_name no)
