File: hardware/VCAT-LightingPCB/canopyBoard/canopyBoard/48PinMCU.kicad_sch (KiCad schematic)
At the start: 34 parts, among them J10 SWD_Header, J11 SWD, SW10 SW_SPDT, SW9 Reset, U10 STM32G473CETx, Y4 Crystal

Commit message: added current check, please dont overwrite my file again
Parts:
- renumbered C68 to C110, C69 to C111, C70 to C112, C71 to C113, C72 to C114, C73 to C115, C74 to C116, C75 to C117, C76 to C118, C77 to C119, C78 to C120, C79 to C121, C80 to C122, C81 to C123, C82 to C124, D22 to D29, D23 to D30, D24 to D31, FB7 to FB11, FB8 to FB12, J10 to J17, J11 to J18, R43 to R63, R44 to R64, R45 to R65, R46 to R70, R47 to R71, R48 to R72, R52 to R73, R53 to R74, SW9 to SW13, SW10 to SW14, U10 to U16, Y4 to Y6
