File: hardware/VCAT-LightingPCB/canopyBoard/canopyBoard/Current Check.kicad_sch (KiCad schematic)
At the start: 8 parts, among them U10 INA180A2, U7 INA180A2, U8 INA180A2, U9 INA180A2

Commit message: please no overrides, complete with bus, hopefully
Connections:
- net GND: now also U8.2 (GND)
- net LEFT_12V: no longer R15.2, U9.4 (-)
- net LEFT_CURR: now also U8.1; no longer U9.1
- net RIGHT_12V: now also R15.2, U9.4 (-); no longer U8.2 (GND)
- net RIGHT_CURR: now also U9.1; no longer U8.1

Commit message: workday, fixed connector logic
Parts:
- removed R12: R, Package_TO_SOT_SMD:SOT-23-5, symbol Device:R
- removed U7: INA180A2, Package_TO_SOT_SMD:SOT-23-5, symbol Amplifier_Current:INA180A2
Connections:
- net STROBE_12V renamed CPY_12V
- net STROBE_CURR renamed CPY_CURR

Commit message: pray for no errors, more stuff to add
Parts:
- R13, R15, R16: value R -> 100m
Other:
- moved on the sheet: R13, R15, R16, U10, U8, U9
