File: hardware/VCAT-LightingPCB/canopyBoard/canopyBoard/Fet Logic.kicad_sch (KiCad schematic)
At the start: 5 parts

Commit message: added current check, please dont overwrite my file again
Parts:
- added IRLML0030TRPBF7: IRLML0030, SOT95P237X112-3N, symbol Transistor_FET:IRLML0030
Connections:
- net GND: now also IRLML0030TRPBF7.2 (S)
- new net STROBE_FET: IRLML0030TRPBF7.3 (D)
- new net STROBE_SIG: IRLML0030TRPBF7.1 (G)
Changed lines of the file:
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@@
+	(wire
+		(pts
+			(xy 116.84 21.59) (xy 116.84 22.86)
+		)
+		(stroke
+			(width 0)
+			(type default)
+		)
+	)
 	(wire
 		(pts
@@
 	(wire
 		(pts
+			(xy 123.19 30.48) (xy 121.92 30.48)
+		)
+		(stroke
+			(width 0)
+			(type default)
+		)
+	)
+	(wire
+		(pts
 			(xy 88.9 57.15) (xy 87.63 57.15)
 		)
@@
 	(wire
 		(pts
+			(xy 110.49 30.48) (xy 111.76 30.48)
+		)
+		(stroke
+			(width 0)
+			(type default)
+		)
+	)
+	(wire
+		(pts
 			(xy 35.56 31.75) (xy 36.83 31.75)
 		)
@@
 		)
 	)
+	(hierarchical_label "GND"
+		(shape input)
+		(at 123.19 30.48 0)
+		(effects
+			(font
+				(size 1.27 1.27)
+			)
+			(justify left)
+		)
+	)
+	(hierarchical_label "STROBE_SIG"
+		(shape input)
+		(at 116.84 21.59 0)
+		(effects
+			(font
+				(size 1.27 1.27)
+			)
+			(justify left)
+		)
+	)
 	(hierarchical_label "RIGHT_FET"
 		(shape input)
@@
 			)
 			(justify left)
+		)
+	)
+	(hierarchical_label "STROBE_FET"
+		(shape input)
+		(at 110.49 30.48 180)
+		(effects
+			(font
+				(size 1.27 1.27)
+			)
+			(justify right)
 		)
 	)
@@
 					(unit 1)
 				)
+			)
+		)
+	)
+	(symbol
+		(lib_id "Transistor_FET:IRLML0030")
+		(at 116.84 27.94 90)
+		(mirror x)
+		(unit 1)
+		(body_style 1)
+		(exclude_from_sim no)
+		(in_bom yes)
+		(on_board yes)
+		(in_pos_files yes)
+		(dnp no)
+		(property "Reference" "IRLML0030TRPBF7"
+			(at 114.554 25.654 90)
+			(hide yes)
+			(show_name no)
+			(do_not_autoplace no)
+			(effects
+				(font
+					(size 1.27 1.27)
+				)
+				(justify left)
+			)
+		)
+		(property "Value" "IRLML0030"
+			(at 118.1099 34.29 0)
+			(hide yes)
+			(show_name no)
+			(do_not_autoplace no)
+			(effects
+				(font
+					(size 1.27 1.27)
+				)
+				(justify left)
+			)
+		)
+		(property "Footprint" "SOT95P237X112-3N"
+			(at 118.745 33.02 0)
+			(hide yes)
+			(show_name no)
+			(do_not_autoplace no)
+			(effects
+				(font
+					(size 1.27 1.27)
+					(italic yes)
+				)
+				(justify left)
+			)
+		)
+		(property "Datasheet" "https://www.infineon.com/dgdl/irlml0030pbf.pdf?fileId=5546d462533600a401535664773825df"
+			(at 120.65 33.02 0)
+			(hide yes)
+			(show_name no)
+			(do_not_autoplace no)
+			(effects
+				(font
+					(size 1.27 1.27)
+				)
+				(justify left)
+			)
+		)
+		(property "Description" "5.3A Id, 30V Vds, 27mOhm Rds, N-Channel HEXFET Power MOSFET, SOT-23"
+			(at 116.84 27.94 0)
+			(hide yes)
+			(show_name no)
+			(do_not_autoplace no)
+			(effects
+				(font
+					(size 1.27 1.27)
+				)
+			)
+		)
+		(pin "2"
+		)
+		(pin "1"
+		)
+		(pin "3"
+		)
+		(instances
+			(project "canopyBoard"
+				(path "/df5034a6-89e6-4596-8ae4-d16cb76dc299/45d7110a-45d7-4ac6-a29f-e84ce60a44ce"
+					(reference "IRLML0030TRPBF7")
+					(unit 1)
+				)

Commit message: workday, fixed connector logic
Parts:
- removed IRLML0030TRPBF2, IRLML0030TRPBF3, IRLML0030TRPBF4: IRLML0030, SOT95P237X112-3N, symbol Transistor_FET:IRLML0030
Connections:
- net LEFT_FET renamed L_PWRFET
- net RIGHT_FET renamed R_PWRFET
- net STROBE_FET renamed CPY_PWRFET
- net STROBE_SIG renamed CPY_SIG

Commit message: pray for no errors, more stuff to add
Connections:
- net CPY_SIG is gone; now on net CPY_PWRFET: IRLML0030TRPBF7.1 (G)
- net LEFT_SIG is gone; now on net L_PWRFET: IRLML0030TRPBF5.1 (G)
- net RIGHT_SIG is gone; now on net R_PWRFET: IRLML0030TRPBF6.1 (G)
- net CPY_PWRFET: no longer IRLML0030TRPBF7.3 (D)
- net L_PWRFET: no longer IRLML0030TRPBF5.3 (D)
- net R_PWRFET: no longer IRLML0030TRPBF6.3 (D)
- new net CPY_BRK: IRLML0030TRPBF7.3 (D)
- new net L_BRK: IRLML0030TRPBF5.3 (D)
- new net R_BRK: IRLML0030TRPBF6.3 (D)
