File: hardware/VCAT-LightingPCB/canopyBoard/canopyBoard/MCU.kicad_sch (KiCad schematic)
At the start: 6 parts

Commit message: added current check, please dont overwrite my file again
Parts:
- removed D39, D40, D41: LED, symbol Device:LED
- removed R81, R82, R83: 1k, symbol Device:R
- added D42, D43, D44: LED, symbol Device:LED
- added R84, R85, R86: 1k, symbol Device:R
Connections:
- net 48PinMCU4/PB0: now also R84.1
- net 48PinMCU4/PB1: now also R85.1
- net 48PinMCU4/PB2: now also R86.1
- net GND: now also D42.1 (K), D43.1 (K), D44.1 (K)
- new net: D42.2 (A), R84.2
- new net: D44.2 (A), R86.2
- new net: D43.2 (A), R85.2
- no-connect marks 21 -> 17

Commit message: please no overrides, complete with bus, hopefully
Connections:
- no-connect marks 17 -> 18
Other:
- removed sheet USB-C_Connector3
- added sheet USB-C_Connector (USB-C_Connector.kicad_sch)
- sheet 48PinMCU4 ports: added USB_DM, USB_DP; removed PA11, PA12

Commit message: workday, fixed connector logic
Connections:
- no-connect marks 18 -> 15

Commit message: pray for no errors, more stuff to add
Parts:
- D42, D43, D44: p/n (none) -> LTST-C193KGKT-5A
Connections:
- no-connect marks 15 -> 19
Other:
- note added: "34 Timer Pins"
- note added: "Timer"
- moved on the sheet: D42, R84, R85, R86

Commit message: Untrack KiCad .history, convert KiCAD-Sharepoint to a submodule, remove LightsPCB
Other:
- sheet USB-C_Connector ports: added USB_D+, USB_D-; removed USB_DM, USB_DP
Changed lines of the file:
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@@
+	)
+	(no_connect
+		(at 81.28 50.8)
 	)
 	(no_connect
@@
 	)
 	(no_connect
+		(at 81.28 48.26)
+	)
+	(no_connect
 		(at 119.38 69.85)
 	)
@@
 	)
 	(no_connect
-		(at 81.28 50.8)
-	)
-	(no_connect
 		(at 160.02 71.12)
 	)
 	(no_connect
 		(at 119.38 43.18)
-	)
-	(no_connect
-		(at 81.28 48.26)
 	)
 	(no_connect
@@
 	(wire
 		(pts
-			(xy 80.01 59.69) (xy 81.28 59.69)
+			(xy 80.01 53.34) (xy 81.28 53.34)
 		)
 		(stroke
@@
 		)
 	)
+	(label "USB_D-"
+		(at 119.38 48.26 180)
+		(effects
+			(font
+				(size 1.27 1.27)
+			)
+			(justify right bottom)
+		)
+	)
 	(label "L_PWRFET"
 		(at 119.38 33.02 180)
@@
 	(label "CPY_PWRFET"
 		(at 119.38 38.1 180)
+		(effects
+			(font
+				(size 1.27 1.27)
+			)
+			(justify right bottom)
+		)
+	)
+	(label "USB_D+"
+		(at 119.38 50.8 180)
 		(effects
 			(font
@@
 	(hierarchical_label "GND"
 		(shape bidirectional)
-		(at 80.01 59.69 180)
+		(at 80.01 53.34 180)
 		(effects
 			(font
@@
 	(sheet
 		(at 81.28 43.18)
-		(size 21.59 17.78)
+		(size 21.59 12.7)
 		(exclude_from_sim no)
 		(in_bom yes)
@@
 		)
 		(property "Sheetfile" "USB-C_Connector.kicad_sch"
-			(at 81.28 61.5446 0)
+			(at 81.28 56.4646 0)
 			(hide yes)
 			(show_name no)
@@
 		)
 		(property "Author" "Shuopu Wang"
-			(at -36.83 -21.59 0)
+			(at -1.27 0 0)
 			(hide yes)
 			(show_name no)
@@
 		)
 		(property "Date Modified" "9/5/2026"
-			(at -36.83 -21.59 0)
+			(at -1.27 0 0)
 			(hide yes)
 			(show_name no)
@@
 		)
 		(pin "GND" input
-			(at 81.28 59.69 180)
+			(at 81.28 53.34 180)
 			(effects
 				(font
@@
 			)
 		)
-		(pin "USB_DM" bidirectional
+		(pin "USB_D+" bidirectional
+			(at 102.87 50.8 0)
+			(effects
+				(font
+					(size 1.27 1.27)
+				)
+				(justify right)
+			)
+		)
+		(pin "USB_D-" bidirectional
 			(at 102.87 48.26 0)
-			(effects
-				(font
-					(size 1.27 1.27)
-				)
-				(justify right)
-			)
-		)
-		(pin "USB_DP" bidirectional
-			(at 102.87 50.8 0)
 			(effects
 				(font
@@
 			(project "canopyBoard"
 				(path "/df5034a6-89e6-4596-8ae4-d16cb76dc299/9e6894d2-35ee-4054-bbed-0d8e56a2fbc9"
-					(page "9")
-				)
-			)
+					(page "4")
+				)
+			)
